Commit message: Added changes that make things work on Friday - Spot moving. Will verify if all of them are needed before merging to feature/gazebo_sim

File: spot_description/urdf/spot.urdf.xacro (robot description, xacro)
@@ -5,4 +5,5 @@
   <!-- Macros for loading the ROS 2 control tags -->
   <xacro:include filename="$(find spot_description)/urdf/spot.ros2_control.xacro" />
+  <xacro:include filename="$(find spot_description)/urdf/spot.physics.gazebo.xacro" />
   <!-- General parameters -->
   <!-- String that will be prepended to all joints and links-->
@@ -54,3 +55,5 @@
     <xacro:add_cameras prefix="$(arg tf_prefix)" />
   </xacro:if>
+  <!-- Gazebo tags -->
+  <xacro:spot_gazebo_physics />
 </robot>

File: spot_description/urdf/spot_macro.xacro (robot description, xacro)
@@ -80,5 +80,5 @@
             <child link="${tf_prefix}front_left_hip" />
             <limit effort="45" velocity="17.647" lower="-0.78539816339744827899"
-                upper="0.78539816339744827899" />
+                upper="0.78539816339744827899" /> <dynamics damping="1.0" friction="0.2" />
         </joint>
         <xacro:if value="${include_transmissions}">
@@ -120,5 +120,5 @@
             <child link="${tf_prefix}front_left_upper_leg" />
             <limit effort="45" velocity="17.647" lower="-0.89884456477707963539"
-                upper="2.2951079663725435509" />
+                upper="2.2951079663725435509" /> <dynamics damping="1.0" friction="0.2" />
         </joint>
         <xacro:if value="${include_transmissions}">
@@ -166,5 +166,5 @@
             <parent link="${tf_prefix}front_left_upper_leg" />
             <child link="${tf_prefix}front_left_lower_leg" />
-            <limit effort="115" velocity="12.0" lower="-2.7929" upper="-0.254801" />
+            <limit effort="115" velocity="12.0" lower="-2.7929" upper="-0.254801" /> <dynamics damping="1.0" friction="0.2" />
         </joint>
         <xacro:if value="${include_transmissions}">
@@ -200,5 +200,5 @@
             <child link="${tf_prefix}front_right_hip" />
             <limit effort="45" velocity="17.647" lower="-0.78539816339744827899"
-                upper="0.78539816339744827899" />
+                upper="0.78539816339744827899" /> <dynamics damping="1.0" friction="0.2" />
         </joint>
         <xacro:if value="${include_transmissions}">
@@ -240,5 +240,5 @@
             <child link="${tf_prefix}front_right_upper_leg" />
             <limit effort="45" velocity="17.647" lower="-0.89884456477707963539"
-                upper="2.2951079663725435509" />
+                upper="2.2951079663725435509" /> <dynamics damping="1.0" friction="0.2" />
         </joint>
         <xacro:if value="${include_transmissions}">
@@ -286,5 +286,5 @@
             <parent link="${tf_prefix}front_right_upper_leg" />
             <child link="${tf_prefix}front_right_lower_leg" />
-            <limit effort="115" velocity="12.0" lower="-2.7929" upper="-0.247563" />
+            <limit effort="115" velocity="12.0" lower="-2.7929" upper="-0.247563" /> <dynamics damping="1.0" friction="0.2" />
         </joint>
         <xacro:if value="${include_transmissions}">
@@ -320,5 +320,5 @@
             <child link="${tf_prefix}rear_left_hip" />
             <limit effort="45" velocity="17.647" lower="-0.78539816339744827899"
-                upper="0.78539816339744827899" />
+                upper="0.78539816339744827899" /> <dynamics damping="1.0" friction="0.2" />
         </joint>
         <xacro:if value="${include_transmissions}">
@@ -360,5 +360,5 @@
             <child link="${tf_prefix}rear_left_upper_leg" />
             <limit effort="45" velocity="17.647" lower="-0.89884456477707963539"
-                upper="2.2951079663725435509" />
+                upper="2.2951079663725435509" /> <dynamics damping="1.0" friction="0.2" />
         </joint>
         <xacro:if value="${include_transmissions}">
@@ -406,5 +406,5 @@
             <parent link="${tf_prefix}rear_left_upper_leg" />
             <child link="${tf_prefix}rear_left_lower_leg" />
-            <limit effort="115" velocity="12.0" lower="-2.7929" upper="-0.267153" />
+            <limit effort="115" velocity="12.0" lower="-2.7929" upper="-0.267153" /> <dynamics damping="1.0" friction="0.2" />
         </joint>
         <xacro:if value="${include_transmissions}">
@@ -440,5 +440,5 @@
             <child link="${tf_prefix}rear_right_hip" />
             <limit effort="45" velocity="17.647" lower="-0.78539816339744827899"
-                upper="0.78539816339744827899" />
+                upper="0.78539816339744827899" /> <dynamics damping="1.0" friction="0.2" />
         </joint>
         <xacro:if value="${include_transmissions}">
@@ -480,5 +480,5 @@
             <child link="${tf_prefix}rear_right_upper_leg" />
             <limit effort="45" velocity="17.647" lower="-0.89884456477707963539"
-                upper="2.2951079663725435509" />
+                upper="2.2951079663725435509" /> <dynamics damping="1.0" friction="0.2" />
         </joint>
         <xacro:if value="${include_transmissions}">
@@ -526,5 +526,5 @@
             <parent link="${tf_prefix}rear_right_upper_leg" />
             <child link="${tf_prefix}rear_right_lower_leg" />
-            <limit effort="115" velocity="12.0" lower="-2.7929" upper="-0.257725" />
+            <limit effort="115" velocity="12.0" lower="-2.7929" upper="-0.257725" /> <dynamics damping="1.0" friction="0.2" />
         </joint>
         <xacro:if value="${include_transmissions}">

Commit message: Tested by resetting the physics parameters to what they were originally. No chamge, robot still walks. Setting parameters OFF but leaving them as available for users in case we need to use them in the future

File: spot_description/urdf/spot.urdf.xacro (robot description, xacro)
@@ -56,5 +56,5 @@
   </xacro:if>
   <!-- Gazebo tags -->
-  <xacro:spot_gazebo_physics />
+  <!--<xacro:spot_gazebo_physics />-->
   <!-- Gazebo plugins: odom state publisher -->
   <!--<xacro:spot_odometry_publisher />-->

File: spot_description/urdf/spot_macro.xacro (robot description, xacro)
@@ -6,6 +6,9 @@
     gripperless:=false
     custom_gripper_base_link:=''
-			tf_prefix
-			include_transmissions=false">
+    tf_prefix
+    include_transmissions=false
+    leg_damping:='0.0'
+    leg_friction:='0.0'">
+    <!-- 1.0, 0.2. First time it walked we used damping:=1.0 and friction:=0.2. Setting it back to zeros it was still walking -->
         <link name="${tf_prefix}body">
             <visual>
@@ -80,5 +83,6 @@
             <child link="${tf_prefix}front_left_hip" />
             <limit effort="45" velocity="17.647" lower="-0.78539816339744827899"
-                upper="0.78539816339744827899" /> <dynamics damping="1.0" friction="0.2" />
+                upper="0.78539816339744827899" />
+            <dynamics damping="${leg_damping}" friction="${leg_friction}" />
         </joint>
         <xacro:if value="${include_transmissions}">
@@ -120,5 +124,6 @@
             <child link="${tf_prefix}front_left_upper_leg" />
             <limit effort="45" velocity="17.647" lower="-0.89884456477707963539"
-                upper="2.2951079663725435509" /> <dynamics damping="1.0" friction="0.2" />
+                upper="2.2951079663725435509" />
+            <dynamics damping="${leg_damping}" friction="${leg_friction}" />
         </joint>
         <xacro:if value="${include_transmissions}">
@@ -166,5 +171,6 @@
             <parent link="${tf_prefix}front_left_upper_leg" />
             <child link="${tf_prefix}front_left_lower_leg" />
-            <limit effort="115" velocity="12.0" lower="-2.7929" upper="-0.254801" /> <dynamics damping="1.0" friction="0.2" />
+            <limit effort="115" velocity="12.0" lower="-2.7929" upper="-0.254801" />
+            <dynamics damping="${leg_damping}" friction="${leg_friction}" />
         </joint>
         <xacro:if value="${include_transmissions}">
@@ -200,5 +206,6 @@
             <child link="${tf_prefix}front_right_hip" />
             <limit effort="45" velocity="17.647" lower="-0.78539816339744827899"
-                upper="0.78539816339744827899" /> <dynamics damping="1.0" friction="0.2" />
+                upper="0.78539816339744827899" />
+            <dynamics damping="${leg_damping}" friction="${leg_friction}" />
         </joint>
         <xacro:if value="${include_transmissions}">
@@ -240,5 +247,6 @@
             <child link="${tf_prefix}front_right_upper_leg" />
             <limit effort="45" velocity="17.647" lower="-0.89884456477707963539"
-                upper="2.2951079663725435509" /> <dynamics damping="1.0" friction="0.2" />
+                upper="2.2951079663725435509" />
+            <dynamics damping="${leg_damping}" friction="${leg_friction}" />
         </joint>
         <xacro:if value="${include_transmissions}">
@@ -286,5 +294,6 @@
             <parent link="${tf_prefix}front_right_upper_leg" />
             <child link="${tf_prefix}front_right_lower_leg" />
-            <limit effort="115" velocity="12.0" lower="-2.7929" upper="-0.247563" /> <dynamics damping="1.0" friction="0.2" />
+            <limit effort="115" velocity="12.0" lower="-2.7929" upper="-0.247563" />
+            <dynamics damping="${leg_damping}" friction="${leg_friction}" />
         </joint>
         <xacro:if value="${include_transmissions}">
@@ -320,5 +329,6 @@
             <child link="${tf_prefix}rear_left_hip" />
             <limit effort="45" velocity="17.647" lower="-0.78539816339744827899"
-                upper="0.78539816339744827899" /> <dynamics damping="1.0" friction="0.2" />
+                upper="0.78539816339744827899" />
+            <dynamics damping="${leg_damping}" friction="${leg_friction}" />
         </joint>
         <xacro:if value="${include_transmissions}">
@@ -360,5 +370,6 @@
             <child link="${tf_prefix}rear_left_upper_leg" />
             <limit effort="45" velocity="17.647" lower="-0.89884456477707963539"
-                upper="2.2951079663725435509" /> <dynamics damping="1.0" friction="0.2" />
+                upper="2.2951079663725435509" />
+            <dynamics damping="${leg_damping}" friction="${leg_friction}" />
         </joint>
         <xacro:if value="${include_transmissions}">
@@ -406,5 +417,6 @@
             <parent link="${tf_prefix}rear_left_upper_leg" />
             <child link="${tf_prefix}rear_left_lower_leg" />
-            <limit effort="115" velocity="12.0" lower="-2.7929" upper="-0.267153" /> <dynamics damping="1.0" friction="0.2" />
+            <limit effort="115" velocity="12.0" lower="-2.7929" upper="-0.267153" />
+            <dynamics damping="${leg_damping}" friction="${leg_friction}" />
         </joint>
         <xacro:if value="${include_transmissions}">
@@ -440,5 +452,6 @@
             <child link="${tf_prefix}rear_right_hip" />
             <limit effort="45" velocity="17.647" lower="-0.78539816339744827899"
-                upper="0.78539816339744827899" /> <dynamics damping="1.0" friction="0.2" />
+                upper="0.78539816339744827899" />
+            <dynamics damping="${leg_damping}" friction="${leg_friction}" />
         </joint>
         <xacro:if value="${include_transmissions}">
@@ -480,5 +493,6 @@
             <child link="${tf_prefix}rear_right_upper_leg" />
             <limit effort="45" velocity="17.647" lower="-0.89884456477707963539"
-                upper="2.2951079663725435509" /> <dynamics damping="1.0" friction="0.2" />
+                upper="2.2951079663725435509" />
+            <dynamics damping="${leg_damping}" friction="${leg_friction}" />
         </joint>
         <xacro:if value="${include_transmissions}">
@@ -526,5 +540,6 @@
             <parent link="${tf_prefix}rear_right_upper_leg" />
             <child link="${tf_prefix}rear_right_lower_leg" />
-            <limit effort="115" velocity="12.0" lower="-2.7929" upper="-0.257725" /> <dynamics damping="1.0" friction="0.2" />
+            <limit effort="115" velocity="12.0" lower="-2.7929" upper="-0.257725" />
+            <dynamics damping="${leg_damping}" friction="${leg_friction}" />
         </joint>
         <xacro:if value="${include_transmissions}">
