Commit message: Robot has a ground truth pose publisher from gazebo

File: spot_description/urdf/spot.ros2_control.xacro (robot description, xacro)
@@ -139,10 +139,10 @@
         <!-- Gazebo ROS Control plugin -->
         <xacro:if value="${interface_type == 'gazebo'}">
-+          <gazebo>
-+            <plugin name="gz_ros2_control::GazeboSimROS2ControlPlugin" filename="gz_ros2_control-system">
-+              <parameters>$(find spot_description)/config/ros2_control_spot.yaml</parameters>
-+          </plugin>
-+          </gazebo>
-+        </xacro:if>
+          <gazebo>
+            <plugin name="gz_ros2_control::GazeboSimROS2ControlPlugin" filename="gz_ros2_control-system">
+              <parameters>$(find spot_description)/config/ros2_control_spot.yaml</parameters>
+          </plugin>
+          </gazebo>
+        </xacro:if>
     </xacro:macro>
 </robot>

File: spot_description/urdf/spot.sensors.gazebo.xacro (robot description, xacro)
@@ -110,3 +110,26 @@
       <xacro:fixed_joint name="camera_back_j" parent="${prefix}base_link" child="${prefix}camera_back" xyz="-0.425 0 0.01" rpy="0 0.3 ${-pi}" />
     </xacro:macro>
+    <!-- Odometry simulation -->
+    <xacro:macro name="spot_odometry_publisher">
+      <gazebo>
+        <plugin filename="gz-sim-odometry-publisher-system" name="gz::sim::systems::OdometryPublisher">
+          <odom_frame>odom</odom_frame>
+          <robot_base_frame>base_link</robot_base_frame>
+          <odom_publish_frequency>10</odom_publish_frequency>
+          <tf_topic>spot/odom</tf_topic>
+        </plugin>
+      </gazebo>
+    </xacro:macro>
+    <!-- PosePublisher - P3D-equivalent -->
+    <xacro:macro name="spot_pose_publisher">
+      <gazebo>
+        <plugin filename="gz-sim-pose-publisher-system" name="gz::sim::systems::PosePublisher">
+          <publish_link_pose>false</publish_link_pose>
+          <publish_nested_model_pose>true</publish_nested_model_pose>
+          <publish_model_pose>true</publish_model_pose>
+          <update_frequency>30</update_frequency>
+          <use_pose_vector_msg>false</use_pose_vector_msg>
+        </plugin>
+      </gazebo>
+    </xacro:macro>
 </robot>

File: spot_description/urdf/spot.urdf.xacro (robot description, xacro)
@@ -57,3 +57,7 @@
   <!-- Gazebo tags -->
   <xacro:spot_gazebo_physics />
+  <!-- Gazebo plugins: odom state publisher -->
+  <!--<xacro:spot_odometry_publisher />-->
+  <!-- Gazebo plugins: pose publisher -->
+  <xacro:spot_pose_publisher />
 </robot>

Commit message: Support frame names with tf_prefix and add camera_info topics

File: spot_description/urdf/spot.ros2_control.xacro (robot description, xacro)
@@ -83,5 +83,5 @@
         </sensor>
     </xacro:macro>
-    <xacro:macro name="spot_ros2_control" params="interface_type has_arm leasing hostname port certificate username password tf_prefix k_q_p k_qd_p">
+    <xacro:macro name="spot_ros2_control" params="interface_type has_arm leasing hostname port certificate username password tf_prefix k_q_p k_qd_p controllers_config">
         <!-- Currently implements a simple system interface that covers all joints of the robot -->
         <ros2_control name="SpotSystem" type="system">
@@ -158,11 +158,11 @@
         </ros2_control>
         <!-- Gazebo ROS Control plugin -->
-        <xacro:if value="${interface_type == 'gazebo'}">
-          <gazebo>
-            <plugin name="gz_ros2_control::GazeboSimROS2ControlPlugin" filename="gz_ros2_control-system">
-              <parameters>$(find spot_description)/config/ros2_control_spot.yaml</parameters>
-          </plugin>
-          </gazebo>
-        </xacro:if>
+                <xacro:if value="${interface_type == 'gazebo'}">
+                    <gazebo>
+                        <plugin name="gz_ros2_control::GazeboSimROS2ControlPlugin" filename="gz_ros2_control-system">
+                            <parameters>${controllers_config}</parameters>
+                        </plugin>
+                    </gazebo>
+                </xacro:if>
     </xacro:macro>
 </robot>

File: spot_description/urdf/spot.sensors.gazebo.xacro (robot description, xacro)
@@ -44,4 +44,5 @@
                     <visualize>${visualize}</visualize>
                     <camera>
+                        <camera_info_topic>${name}_fisheye/camera_info</camera_info_topic>
                         <horizontal_fov>${radians(102.35)}</horizontal_fov> <!-- computed from real fx -->
                         <image>
@@ -76,4 +77,5 @@
                     <topic>${name}_depth</topic>
                     <camera>
+                        <camera_info_topic>${name}_depth/camera_info</camera_info_topic>
                         <horizontal_fov>${radians(102.35)}</horizontal_fov> <!-- put here equal to mono cam -->
                         <optical_frame_id>${prefix}camera_${name}</optical_frame_id>
@@ -100,7 +102,7 @@
     <xacro:macro name="add_cameras" params="prefix:='' ">
       <xacro:spot_camera prefix="${prefix}" name="frontleft" simulate="1" />
-      <xacro:fixed_joint name="camera_frontleft_j" parent="${prefix}base_link" child="${prefix}camera_frontleft" xyz="0.415 0.037 -0.01" rpy="0.0 0.353917 -0.554196" /> <!-- r: 1.355558 -->
+      <xacro:fixed_joint name="camera_frontleft_j" parent="${prefix}base_link" child="${prefix}camera_frontleft" xyz="0.415 0.037 -0.01" rpy="0.0 0.353917 -0.554196" /> <!-- r 1.355558 -->
       <xacro:spot_camera prefix="${prefix}" name="frontright" simulate="1" />
-      <xacro:fixed_joint name="camera_frontright_j" parent="${prefix}base_link" child="${prefix}camera_frontright" xyz="0.415 -0.037 -0.01" rpy="0.0 0.353917 0.554196" /> <!-- r: -1.355558-->
+      <xacro:fixed_joint name="camera_frontright_j" parent="${prefix}base_link" child="${prefix}camera_frontright" xyz="0.415 -0.037 -0.01" rpy="0.0 0.353917 0.554196" /> <!-- r -1.355558-->
       <xacro:spot_camera prefix="${prefix}" name="left" simulate="1" />
       <xacro:fixed_joint name="camera_left_j" parent="${prefix}base_link" child="${prefix}camera_left" xyz="-0.125 0.12 0.035" rpy="0 0.2 ${pi/2}" />

File: spot_description/urdf/spot.urdf.xacro (robot description, xacro)
@@ -7,6 +7,8 @@
   <xacro:include filename="$(find spot_description)/urdf/spot.physics.gazebo.xacro" />
   <!-- General parameters -->
-  <!-- String that will be prepended to all joints and links-->
+  <!-- String that will be prepended to all joints and links -->
+  <!-- Primary argument: tf_prefix. Alias: prefix (for compatibility). If both are set, they will be concatenated. -->
   <xacro:arg name="tf_prefix" default="" />
+  <xacro:arg name="prefix" default="" />
   <!-- Set to true if Spot has an arm -->
   <xacro:arg name="arm" default="false" />
@@ -29,9 +31,11 @@
   <!-- Simulate cameras -->
   <xacro:arg name="simulate_cameras" default="True" />
+  <!-- Path to ros2_control controllers config (YAML). Defaults to this package's config. -->
+  <xacro:arg name="controllers_config" default="$(find spot_description)/config/ros2_control_spot.yaml" />
   <!-- Load Spot -->
   <xacro:load_spot
     arm="$(arg arm)"
     feet="$(arg feet)"
-    tf_prefix="$(arg tf_prefix)"
+    tf_prefix="$(arg tf_prefix)$(arg prefix)"
     gripperless="$(arg gripperless)"
 	  include_transmissions="$(arg include_transmissions)" />
@@ -46,18 +50,19 @@
                                username="$(arg username)"
                                password="$(arg password)"
-                               tf_prefix="$(arg tf_prefix)"
+               tf_prefix="$(arg tf_prefix)$(arg prefix)"
                                k_q_p="$(arg k_q_p)"
-                               k_qd_p="$(arg k_qd_p)" />
+               k_qd_p="$(arg k_qd_p)"
+               controllers_config="$(arg controllers_config)" />
   </xacro:if>
   <!-- Adding cameras -->
   <xacro:if value="$(arg simulate_cameras)">
     <xacro:include filename="$(find spot_description)/urdf/spot.sensors.gazebo.xacro" />
-    <xacro:add_cameras prefix="$(arg tf_prefix)" />
+    <xacro:add_cameras prefix="$(arg tf_prefix)$(arg prefix)" />
   </xacro:if>
   <!-- Gazebo tags -->
   <!--<xacro:spot_gazebo_physics />-->
-  <!-- Gazebo plugins: odom state publisher -->
+  <!-- Gazebo plugins odom state publisher -->
   <!--<xacro:spot_odometry_publisher />-->
-  <!-- Gazebo plugins: pose publisher -->
+  <!-- Gazebo plugins pose publisher -->
   <xacro:spot_pose_publisher />
 </robot>
